Commit message: REP Inv kinematics update

File: tesseract/tesseract_support/urdf/abb_irb2400_external_positioner.urdf (robot description, URDF)
Before this commit: robot abb_irb2400_external_positioner, 12 links, 11 joints
Links:
- added link positioner_link_1
Joints:
- added joint positioner_joint_2: type prismatic, parent positioner_link_1, child positioner_tool0, origin xyz=0 0 0 rpy=0 0 0, axis 1 0 0, limit lower=-1.0 upper=1.0 effort=0 velocity=2.618
- joint positioner_joint_1: child positioner_tool0 -> positioner_link_1

File: tesseract_ros_workcell/twc_support/CAD/eoat/ati_9120_tsm_mmb_8432/urdf/ati_9120_tsm_mmb_8432_macro.xacro (robot description, xacro)
@@ -18,10 +18,17 @@
     </link>
     <link name="${prefix}tool0"/>
+    <link name="${prefix}dock"/>
     <!-- end of link list -->
     <!-- joint list -->
     <joint name="${prefix}base_link_tool0" type="fixed">
-      <origin xyz="0 0.05398 0.01524" rpy="0 0 0" />
+      <origin xyz="0 0 0.03048" rpy="0 0 0" />
       <parent link="${prefix}base_link" />
       <child link="${prefix}tool0" />
+    </joint>
+    <!-- joint list -->
+    <joint name="${prefix}base_link_dock" type="fixed">
+      <origin xyz="-0.09108 0 0.14835" rpy="-1.5708 0 -1.5708" />
+      <parent link="${prefix}tool0" />
+      <child link="${prefix}dock" />
     </joint>
     <!-- end of joint list -->

File: tesseract_ros_workcell/twc_support/urdf/workcell_positioner_macro.xacro (robot description, xacro)
@@ -35,6 +35,5 @@
     <xacro:ros_industrial_logo prefix="logo_"/>
     <!-- link list -->
-    <link name="${prefix}world" />
-    <link name="${prefix}tool_dock0" />
+    <link name="${prefix}world"/>
     <link name="${prefix}part_link">
       <visual>
@@ -58,5 +57,5 @@
     </joint>
     <joint name="${prefix}world_pedestal_joint" type="fixed">
-      <origin xyz="0 -1 0" rpy="0 0 1.5708" />
+      <origin xyz="0 -1.5 0" rpy="0 0 1.5708" />
       <parent link="${prefix}world" />
       <child link="${prefix}pedestal_base_link" />
@@ -88,9 +87,4 @@
       <child link="${prefix}ati_qc110m_base_link" />
     </joint>
-    <joint name="${prefix}world_tool_dock0_joint" type="fixed">
-      <origin xyz="-1 -1 1" rpy="-1.5708 -1.5708 -3.14" />
-      <parent link="${prefix}world" />
-      <child link="${prefix}tool_dock0" />
-    </joint>
     <!--<joint name="${prefix}tool_dock0_ati_f_joint" type="fixed">
       <origin xyz="0 0 0" rpy="0 0 0" />
@@ -120,5 +114,5 @@
     <joint name="${prefix}positioner_part_joint" type="fixed">
 <!--      <origin xyz="-0.4 -1.1 -0.2" rpy="0 -0.523599 0" />-->
-      <origin xyz="-0.55 -1.1 0" rpy="0 0 0" />
+      <origin xyz="-0.55 -1.1 -0.2" rpy="0 0 0" />
       <parent link="${prefix}positioner_tool0" />
       <child link="${prefix}part_link" />
