Commit message: One point trajopt

File: abb_example/urdf/m1_workcell.xacro (robot description, xacro)
@@ -1,4 +1,4 @@
 <?xml version="1.0" ?>
-<robot name="puzzle_piece_workcell" xmlns:xacro="http://wiki.ros.org/xacro">
+<robot name="m1_workcell" xmlns:xacro="http://wiki.ros.org/xacro">
   <!-- This contains the macro "ses_part_macro" that places the clip wrt the tool tip -->
   <xacro:include filename="$(find twc_support)/CAD/robot/abb_irbpa250_d1000/urdf/irbpa250_d1000_macro.xacro"/>
@@ -15,5 +15,5 @@
     <parent link="world"/>
     <child link="base_link"/>
-    <origin xyz="0 0 0" rpy="0 0 0"/>
+    <origin xyz="1.8 0 1.2" rpy="0 0 3.14"/>
   </joint>
 </robot>

Commit message: working ext_axis

File: abb_example/urdf/m1_workcell.xacro (robot description, xacro)
@@ -15,5 +15,5 @@
     <parent link="world"/>
     <child link="base_link"/>
-    <origin xyz="0 0 0" rpy="0 0 0"/>
+    <origin xyz="1.8 0 1.2" rpy="0 0 3.14"/>
   </joint>
 </robot>

Commit message: four points linear raster

File: abb_example/urdf/m1_workcell.xacro (robot description, xacro)
@@ -7,4 +7,10 @@
   <xacro:abb_irb2600_12_165 prefix=""/>
   <link name="world"/>
+  <link name="pos_too0_viz"/>
+  <joint name="visulizer" type="fixed">
+    <parent link="positioner_tool0"/>
+    <child link="pos_too0_viz"/>
+    <origin xyz="0 0 0" rpy="0 0 0"/>
+  </joint>
   <joint name="world_to_positioner" type="fixed">
     <parent link="world"/>
